File: pcb/meterbus_frontend.kicad_sch (KiCad schematic)
At the start: 34 parts, among them Q1 2N7002, U1 78L05G, U3 ISO6721RBDR, U5 74HC14D

Commit message: lib: move customized JLCPCB symbols into custom library
Three JLCPCB symbols had pin electrical types edited in place in the
vendored subtree, which the subtree drift check rejects. Copy them into
custom_symbols under their MPNs, repoint the schematic, and restore the
subtree to its recorded squash commit.

  X1  Crystal, 32.768kHz, 13pF   -> custom_symbols:Q13FC1350000400
  D7  TVS-Bi, PSM712-LF-T7       -> custom_symbols:PSM712-LF-T7
  U1  LDO, 5V, 0.1A              -> custom_symbols:78L05G

Pin geometry is unchanged, so existing wiring is unaffected. The fourth
edited symbol, LDO, 3.3V, 0.1A (HT7533), is no longer used by the board
and was dropped rather than copied.

Co-Authored-By: Claude Opus 5 <noreply@anthropic.com>
Parts:
- D7: symbol PCM_JLCPCB-Diode-Packages:TVS-Bi, PSM712-LF-T7 -> custom_symbols:PSM712-LF-T7
- U1: symbol PCM_JLCPCB-Power:LDO, 5V, 0.1A -> custom_symbols:78L05G
Changed lines of the file:
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@@
 	)
 	(symbol
-		(lib_id "PCM_JLCPCB-Power:LDO, 5V, 0.1A")
+		(lib_id "custom_symbols:78L05G")
 		(at 66.04 96.52 0)
 		(unit 1)
@@
 	)
 	(symbol
-		(lib_id "PCM_JLCPCB-Diode-Packages:TVS-Bi, PSM712-LF-T7")
+		(lib_id "custom_symbols:PSM712-LF-T7")
 		(at 73.66 46.99 270)
 		(unit 1)
