File: pcb/mcu.kicad_sch (KiCad schematic)
At the start: 27 parts, among them J2 DEBUG, U7 ESP32-C6-WROOM-1-N8, X1 Q13FC1350000400

Commit message: sch: rewire SPI to supply separate clock lines to flash and ethernet
The flash IC datasheet specifies that the SPI clock must not be toggled
while CS is high, which means we need to separate the ethernet and flash
clock lines.

I've GPIO3 on the ESP for the flash clock line, and plan to use the
internal peripheral MUX to switch it when talking with the IC.

I've also moved a bunch of test points and termination resistors in this
process.
Parts:
- removed R56: 33Ω, PCM_JLCPCB:R_0603, symbol PCM_JLCPCB-Resistors:0603,33Ω
- removed TP4: SCK, TestPoint:TestPoint_Pad_D1.0mm, symbol Connector:TestPoint_Square
- removed TP7: MOSI, TestPoint:TestPoint_Pad_D1.0mm, symbol Connector:TestPoint_Square
- removed TP8: MISO, TestPoint:TestPoint_Pad_D1.0mm, symbol Connector:TestPoint_Square
- removed TP9: GND, TestPoint:TestPoint_Plated_Hole_D2.0mm, symbol Connector:TestPoint_Square
- added NT2, NT3: NetTie_3_Tee, symbol Device:NetTie_3_Tee
- added R62, R63, R64, R65: 33Ω, PCM_JLCPCB:R_0603, symbol PCM_JLCPCB-Resistors:0603,33Ω
- added TP16: MISO, TestPoint:TestPoint_Pad_D1.0mm, symbol Connector:TestPoint_Square
- added TP32: GND, TestPoint:TestPoint_Plated_Hole_D2.0mm, symbol Connector:TestPoint_Square
- added TP34: MOSI, TestPoint:TestPoint_Pad_D1.0mm, symbol Connector:TestPoint_Square
Connections:
- net GND: now also TP32.1
- net MCU_MOSI: now also R65.1, TP34.1
- net MCU_FLASH_SCK: now reaches U7.26 (IO3)
- net MCU_FLASH_SCK: now also R64.1
- net ETH_CS renamed ETH.CS
- net ETH.CS: now also R62.2; no longer U7.16 (IO18)
- net FLASH_CS renamed FLASH.CS
- net FLASH.CS: now also R63.2; no longer U7.17 (IO19)
- net MCU_SCK renamed MCU_ETH_SCK
- net MISO renamed MCU_MISO
- net MCU_MISO: now also NT3.3, TP16.1
- net SCK renamed ETH.SCK
- new net: NT2.3, R65.2
- new net ETH.MISO: NT3.2
- new net ETH.MOSI: NT2.2
- new net FLASH.MISO: NT3.1
- new net FLASH.MOSI: NT2.1
- new net FLASH.SCK: R64.2
- new net MCU_ETH_CS: R62.1, U7.16 (IO18)
- new net MCU_FLASH_CS: R63.1, U7.17 (IO19)
- no-connect marks 3 -> 2
Other:
- note added: "The flash IC specifies that the SPI clock line must not be toggled while CS is high, meaning separate clock lines are needed for each device in addition to separate CS lines."
- moved on the sheet: R55

Commit message: sch: increase bulk bypass capacitance for ESP32
WiFi tx and other intensive operations can chug a bit of current, so
increase to 22uF
Parts:
- removed C15: 10uF, PCM_JLCPCB:C_0603, symbol PCM_JLCPCB-Capacitors:0603,10uF,(2)
- added C8: 22uF, PCM_JLCPCB:C_0603, symbol PCM_JLCPCB-Capacitors:0603,22uF
Connections:
- net +3V3: now also C8.2
- net GND: now also C8.1
