File: pcb/mcu.kicad_sch (KiCad schematic)
At the start: 31 parts, among them J2 DEBUG, U7 ESP32-C6-WROOM-1-N8, X1 Q13FC1350000400

Commit message: lib: move customized JLCPCB symbols into custom library
Three JLCPCB symbols had pin electrical types edited in place in the
vendored subtree, which the subtree drift check rejects. Copy them into
custom_symbols under their MPNs, repoint the schematic, and restore the
subtree to its recorded squash commit.

  X1  Crystal, 32.768kHz, 13pF   -> custom_symbols:Q13FC1350000400
  D7  TVS-Bi, PSM712-LF-T7       -> custom_symbols:PSM712-LF-T7
  U1  LDO, 5V, 0.1A              -> custom_symbols:78L05G

Pin geometry is unchanged, so existing wiring is unaffected. The fourth
edited symbol, LDO, 3.3V, 0.1A (HT7533), is no longer used by the board
and was dropped rather than copied.

Co-Authored-By: Claude Opus 5 <noreply@anthropic.com>
Parts:
- X1: symbol PCM_JLCPCB-Crystals:Crystal, 32.768kHz, 13pF -> custom_symbols:Q13FC1350000400
Changed lines of the file:
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@@
 	)
 	(symbol
-		(lib_id "PCM_JLCPCB-Crystals:Crystal, 32.768kHz, 13pF")
+		(lib_id "custom_symbols:Q13FC1350000400")
 		(at 264.16 146.05 0)
 		(unit 1)
@@
 		)
 		(property "Datasheet" "https://www.lcsc.com/datasheet/lcsc_datasheet_2404180925_Seiko-Epson-Q13FC13500004_C32346.pdf"
-			(at 261.874 145.923 0)
+			(at 249.174 153.924 0)
 			(hide yes)
 			(show_name no)
@@
 		)
 		(property "Description" "-40°C~+85°C 12.5pF 32.768kHz 70kΩ Crystal Oscillator ±20ppm SMD3215-2P Crystals ROHS"
-			(at 264.16 146.05 0)
+			(at 264.16 151.892 0)
 			(hide yes)
 			(show_name no)
@@
 		)
 		(property "LCSC" "C32346"
-			(at 264.16 146.05 0)
+			(at 263.906 133.096 0)
 			(hide yes)
 			(show_name no)
@@
 		)
 		(property "Stock" "614447"
-			(at 264.16 146.05 0)
+			(at 264.16 123.952 0)
 			(hide yes)
 			(show_name no)
@@
 		)
 		(property "Price" "0.168USD"
-			(at 264.16 146.05 0)
+			(at 264.16 131.318 0)
 			(hide yes)
 			(show_name no)
@@
 		)
 		(property "Process" "SMT"
-			(at 264.16 146.05 0)
+			(at 265.176 120.396 0)
 			(hide yes)
 			(show_name no)
@@
 		)
 		(property "Class" "Basic Component"
-			(at 264.16 146.05 0)
+			(at 264.668 140.716 0)
 			(hide yes)
 			(show_name no)
@@
 		)
 		(property "Category" "Crystals/Oscillators/Resonators,Crystals"
-			(at 264.16 146.05 0)
+			(at 264.668 150.368 0)
 			(hide yes)
 			(show_name no)
@@
 		)
 		(property "Manufacturer" "Seiko Epson"
-			(at 264.16 146.05 0)
+			(at 264.668 125.73 0)
 			(hide yes)
 			(show_name no)
@@
 		)
 		(property "Part" "Q13FC13500004"
-			(at 264.16 146.05 0)
+			(at 264.922 127.762 0)
 			(hide yes)
 			(show_name no)
@@
 		)
 		(property "Frequency" "32.768kHz"
-			(at 264.16 146.05 0)
+			(at 264.16 137.16 0)
 			(hide yes)
 			(show_name no)
@@
 		)
 		(property "Equivalent Series Resistance (Esr)" "70kΩ"
-			(at 264.16 146.05 0)
+			(at 264.16 138.938 0)
 			(hide yes)
 			(show_name no)
@@
 		)
 		(property "Operating Temperature" "-40°C~+85°C"
-			(at 264.16 146.05 0)
+			(at 264.16 129.286 0)
 			(hide yes)
 			(show_name no)
@@
 		)
 		(property "Frequency Tolerance" "±20ppm"
-			(at 264.16 146.05 0)
+			(at 265.43 140.462 0)
 			(hide yes)
 			(show_name no)
@@
 		)
 		(property "Crystal Type" "SMD Crystal Resonator"
-			(at 264.16 146.05 0)
+			(at 264.16 135.382 0)
 			(hide yes)
 			(show_name no)
@@
 		)
 		(property "Load Capacitance" "12.5pF"
-			(at 264.16 146.05 0)
+			(at 265.43 140.462 0)
 			(hide yes)
 			(show_name no)
@@
 		)
 		(property "Normal Temperature Frequency Tolerance" "±20ppm"
-			(at 264.16 146.05 0)
+			(at 264.414 140.462 0)
 			(hide yes)
 			(show_name no)
@@
 		)
 		(property "Equivalent Series Resistance(Esr)" "70kΩ"
-			(at 264.16 146.05 0)
+			(at 264.414 122.174 0)
 			(hide yes)
 			(show_name no)
@@
 		)
 		(property "Type" "Surface Mount Crystal"
-			(at 264.16 146.05 0)
-			(hide yes)
-			(show_name no)
+			(at 265.176 120.396 0)
+			(hide yes)
+			(show_name no)
